File: KiCad schematic + PCB/mouse_pic.kicad_pcb (KiCad board)
At the start: 2 copper layers, 49.8 x 61.7 mm, 71 parts, among them P11 TestPoint, P12 TestPoint, P13 TestPoint, P14 TestPoint, P15 TestPoint, P20 TestPoint, P21 TestPoint, P26 TestPoint, P27 TestPoint, P28 TestPoint, P29 TestPoint, P30 TestPoint, P31 TestPoint, P32 TestPoint, SW1 SW_SPDT, SW2 SW_SPDT, SW3 SW_SPDT, SW4 SW_SPDT, SW5 SW_SPDT, SW6 SW_SPDT, U1 LM1117-1.8V, U10 NCP1117-3.3_SOT223, U2 PMW3360DM-T2QU, U3 RP2040, U4 W25Q32JVSS, Y1 ABM8-272-T3

Commit message: Enhance PMW3360 mouse firmware with improved SROM handling, button mapping, and hardware verification documentation. Added timeout for SPI capture to prevent hangs, updated Readme with runtime controls and settings persistence details, and modified KiCad files for compatibility with newer versions.
Parts:
- R40: value R39 -> 39
